File: eagle/step_motor.sch (EAGLE design)
At the start: 42 parts, among them IC1 LM2937, U1 L6470

Commit message: CHG: Final board version
Parts:
- removed C3: 0.22uF, rcl:C-EUC0603
- removed C4: 100uF, SparkFun-Capacitors:100UF-ELECT
- removed EN800: PEC11R, Radio Projekt:PEC11R
- removed IC1: LM2937, linear:LM2937
- removed R1, R2: 10k, rcl:R-EU_R0603
- removed R4: 200k, SparkFun:POTTRIM
- added C120: 1u, rcl:C-EUC1206
- added C121, C123: 100n, rcl:C-EUC0603
- added C124: 10u, rcl:C-EUC1206
- added C300: 100uF, rcl:CPOL-EUD
- added IC110: UA78M05DCY, linear:UA78M05DCY
- added IC120: (no value), linear-technology:LT1129CS8
- added JP2: (no value), pinhead:PINHD-1X5
- added R120: 91k, rcl:R-EU_R0603
- added R121: 24k, rcl:R-EU_R0603
- added R341: 200k, rcl:R-TRIMM3224X
- added X1: MICROMATCH-4, con-amp-micromatch:MICROMATCH-4
- C310: value 0.1uF -> 100n
- R342: value 8.2k -> 8k2
- renumbered C1 to C310, C10 to C112, C11 to C110, C12 to C113, C13 to C201, C14 to C200, C2 to C311, C5 to C321, C6 to C320, C7 to C330, C8 to C312, C800 to C100, C801 to C101, C802 to C102, C9 to C111, D1 to D320, R3 to R330, R5 to R342, R6 to R340, R7 to R200, R800 to R100, R801 to R101, R802 to R102, R803 to R103, R804 to R104, R805 to R105, S1 to S330, U$4 to IC200, U1 to IC300
Connections:
- net N$7 renamed C320
- removed net ADC: R342.2, R4.A, R4.S
- removed net VCC: C110.1, C111.1, C3.1, C4.+, IC1.VI
- removed net VLOGIC: C310.1, C311.+, R1.2, R2.2
- new net +18V: C123.1, C124.1, IC120G$1.OUT, R120.2, X1-1.S
- new net MSP430_FREE_1: IC200.3
- new net MSP430_FREE_2: IC200.15
- new net N$2: IC120G$1.SENSE, R120.1, R121.1
- new net SDI: IC200.7, X1-2.S
- new net SDO: IC200.6, X1-3.S
- net !L6470_BUSY: now also IC200.16; no longer IC200.15, R1.1
- net !L6470_CS: now also IC200.5; no longer IC200.14
- net !L6470_FLAG: now also IC200.14; no longer IC200.13, R2.1
- net !L6470_RST: now also IC200.11; no longer IC200.12
- net +3V3: now also C310.1, C311.+, IC110.VO; no longer IC1.VO
- net ENCODER_A: now also IC200.21; no longer IC200.9
- net ENCODER_B: now also IC200.22; no longer IC200.10
- net ENCODER_SW: now also IC200.17; no longer IC200.11
- net GND: now also C120.2, C121.2, C123.2, C124.2, IC110.GND, IC110.GND@1, IC120G$1.GND, JP2.2, JP2.4, R121.2, X1-4.S; no longer EN800.C, EN800.W, IC1.GND
- net L6470_ADC: now also R341.A, R341.S, R342.2
- net L6470_OSCIN: now also IC200.19; no longer IC200.6
- net L6470_STCK: now also IC200.13; no longer IC200.16
- net MSP430_CLK: now also IC200.4; no longer IC200.5
- net MSP430_MISO: now also IC200.1; no longer IC200.21
- net MSP430_MOSI: now also IC200.2; no longer IC200.22
- net N$11: now also R341.E; no longer R4.E
- net N$33: now also JP2.3; no longer EN800.A
- net N$36: now also JP2.1; no longer EN800.S
- net PGND: now also C300.-; no longer C3.2, C4.-
- net R904: now also JP2.5; no longer EN800.B
- net VS: now also C110.1, C111.1, C120.1, C121.1, C300.+, IC110.VI, IC120G$1.IN
